File: MCU.kicad_sch (KiCad schematic)
At the start: 33 parts, among them J2 Micro_SD_Card_Det_Hirose_DM3AT, J3 HC-TYPE-C-16P-01A, U3 RP2040, U5 W25Q16JVSS, Y1 RH100-12.000-18-2030-TR

Commit message: Update
Parts:
- added C12: 0u1, Capacitor_SMD:C_0603_1608Metric_Pad1.08x0.95mm_HandSolder, symbol Device:C
- added R13, R14, R15: 43R, symbol Device:R
Connections:
- net +3V3: now also J2.4 (VDD), C12.1
- net GND: now also J2.6 (VSS), C12.2
- net at U3.17 (GPIO14): now also R13.1
- net at U3.18 (GPIO15): now also R14.1
- net SD_SPI_MISO: now reaches U3.27 (GPIO16)
- net SD_SPI_MISO: now also R15.2
- net SD_SPI_CS: now reaches U3.28 (GPIO17)
- net SD_SPI_CS: now also J2.2 (DAT3/CD)
- net SD_DET: now reaches U3.29 (GPIO18)
- net SD_SPI_MOSI: now reaches J2.3 (CMD)
- net SD_SPI_MOSI: now also R14.2
- net SD_SPI_SCK: now reaches J2.5 (CLK)
- net SD_SPI_SCK: now also R13.2
- net at J2.7 (DAT0): now also R15.1
- no-connect marks 2 -> 4
Other:
- moved on the sheet: C15, C16, C17, C18, C19, C20, C21, C22, C23, C24, C25, C26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

Commit message: Add RTC
Parts:
- removed C11: 1n, symbol Device:C
- removed C12: 0u1, Capacitor_SMD:C_0603_1608Metric_Pad1.08x0.95mm_HandSolder, symbol Device:C
- removed J2: Micro_SD_Card_Det_Hirose_DM3AT, Connector_Card:microSD_HC_Hirose_DM3AT-SF-PEJM5, symbol Connector:Micro_SD_Card_Det_Hirose_DM3AT
- removed R12: 100k, symbol Device:R
- removed R15: 43R, symbol Device:R
- added C10, C2, C9: 0u1, Capacitor_SMD:C_0603_1608Metric_Pad1.08x0.95mm_HandSolder, symbol Device:C
- added C35: 1n, Capacitor_SMD:C_0603_1608Metric_Pad1.08x0.95mm_HandSolder, symbol Device:C
- added J9: Conn_ARM_JTAG_SWD_10, Connector_PinHeader_1.27mm:PinHeader_2x05_P1.27mm_Vertical, symbol Connector:Conn_ARM_JTAG_SWD_10
- added R16, R22: 100k, Resistor_SMD:R_0603_1608Metric_Pad0.98x0.95mm_HandSolder, symbol Device:R
- added R17: 5k1, Resistor_SMD:R_0603_1608Metric_Pad0.98x0.95mm_HandSolder, symbol Device:R
- added R18, R19: 10k, Resistor_SMD:R_0603_1608Metric_Pad0.98x0.95mm_HandSolder, symbol Device:R
- added U2: 74LVC2G66, Package_SO:VSSOP-8_2.3x2mm_P0.5mm, symbol 74xGxx:74LVC2G66
- added U7: LM393PWR, Package_SO:TSSOP-8_4.4x3mm_P0.65mm, symbol Comparator:LM393
- added U8: 74AHCT1G08, Package_TO_SOT_SMD:SOT-23-5, symbol 74xGxx:74AHCT1G08
- C8: footprint (none) -> Capacitor_SMD:C_0603_1608Metric_Pad1.08x0.95mm_HandSolder
- R1, R10, R11, R13, R14, R2, R3, R6, R7, R8, R9: footprint (none) -> Resistor_SMD:R_0603_1608Metric_Pad0.98x0.95mm_HandSolder
Connections:
- net SD_SPI_CS is gone; now on net SPI0_EXT_CS1: U3.28 (GPIO17)
- net +3V3: now also J9.1 (VTref)
- net +5V: now also C10.1, C2.1, C9.1, R16.1, R18.2, R19.2, R22.1, U2.8 (VCC), U7.8 (V+), U8.5 (VCC)
- net GND: now also U3.19 (TESTEN), C10.2, C2.2, C35.2, C9.2, J9.3 (GND), J9.5 (GND), R17.2, U2.4 (GND), U7.4 (V-), U8.3 (GND)
- net SD_DET: now also U3.18 (GPIO15); no longer U3.29 (GPIO18)
- net SPI0_EXT_CS1: no longer U3.12 (GPIO9)
- net at U3.14 (GPIO11): now also R14.1
- net SPI1_MISO: now reaches U3.15 (GPIO12)
- net SPI1_SD_CS: now reaches U3.16 (GPIO13)
- net SWCLK: now reaches U3.24 (SWCLK)
- net SWCLK: now also J9.4 (SWDCLK/TCK), U2.2
- net SWD: now reaches U3.25 (SWD)
- net SWD: now also U2.6
- net SW2: now reaches U3.30 (GPIO19)
- net SR_nEN: now reaches U3.31 (GPIO20)
- net SPI0_EXT_CS2: now reaches U3.32 (GPIO21)
- net PWM: now reaches U3.34 (GPIO22)
- net SR_LATCH: now reaches U3.35 (GPIO23)
- net SR_DAT: now reaches U3.36 (GPIO24)
- net SR_CLK: now reaches U3.37 (GPIO25)
- net SW3: now reaches U3.38 (GPIO26_ADC0)
- net SW4: now reaches U3.39 (GPIO27_ADC1)
- net AIN0: now reaches U3.40 (GPIO28_ADC2)
- net AIN1: now reaches U3.41 (GPIO29_ADC3)
- net UC_CC1: now reaches J3.A5 (CC1), R9.1
- net UC_CC1: now also U7.3 (+)
- net SWD_GATED: now reaches J3.A8 (SBU1)
- net SWD_GATED: now also U2.5
- net UC_CC2: now reaches J3.B5 (CC2), R10.1
- net UC_CC2: now also U7.5 (+)
- net SWCLK_GATED: now reaches J3.B8 (SBU2)
- net SWCLK_GATED: now also U2.1
- net SD_SPI_MISO renamed RTC_INT
- net SD_SPI_MOSI renamed SPI1_MOSI
- net SD_SPI_SCK renamed SPI1_SCK
- net rst renamed RST
- net RST: now also C35.1, J9.10 (~{RESET}), R22.2
- new net CC1_DET: R18.1, U7.1, U8.1
- new net CC2_DET: R19.1, U7.7, U8.2
- new net SPI1_RTC_CS: U3.12 (GPIO9)
- new net SW1: U3.29 (GPIO18)
- new net SWDIO: J9.2 (SWDIO/TMS)
- new net USBC_CC_THRES: R16.2, R17.1, U7.2 (-), U7.6 (-)
- new net USBC_DAM: U2.3, U2.7, U8.4
- no-connect marks 4 -> 3
Other:
- moved on the sheet: C15, C16, C17, C18, C19, C20, C21, C22, C23, C24, C25, C26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

Commit message: Begin layout
Parts:
- removed C25: 0u1, Capacitor_SMD:C_0603_1608Metric_Pad1.08x0.95mm_HandSolder, symbol Device:C
- added R25, R26: 22R, Resistor_SMD:R_0603_1608Metric_Pad0.98x0.95mm_HandSolder, symbol Device:R
Connections:
- net SWDIO is gone; now on net SWD: J9.2 (SWDIO/TMS)
- net USB_D+: now also R25.1; no longer U3.47 (USB_DP)
- net USB_D-: now also R26.1; no longer U3.46 (USB_DM)
- new net: R26.2, U3.46 (USB_DM)
- new net: R25.2, U3.47 (USB_DP)
Other:
- moved on the sheet: C2, U7C

Commit message: Update layout
Parts:
- removed R18, R19: 10k, Resistor_SMD:R_0603_1608Metric_Pad0.98x0.95mm_HandSolder, symbol Device:R
- removed U7: LM393PWR, Package_SO:TSSOP-8_4.4x3mm_P0.65mm, symbol Comparator:LM393
- removed U8: 74AHCT1G08, Package_TO_SOT_SMD:SOT-23-5, symbol 74xGxx:74AHCT1G08
- added C45: 0u1, Capacitor_SMD:C_0603_1608Metric_Pad1.08x0.95mm_HandSolder, symbol Device:C
- added C46: 1u, Capacitor_SMD:C_0805_2012Metric_Pad1.18x1.45mm_HandSolder, symbol Device:C
- added U11: MAX6106, Package_TO_SOT_SMD:SOT-23, symbol Reference_Voltage:MAX6106
- added U7: TLV7012, Package_TO_SOT_SMD:TSOT-23-8, symbol Global:TLV7012
- added U8: 74LVC1G08, Package_TO_SOT_SMD:SOT-23-5, symbol Global:SN74LV1T08
- C27, C28: value 27p -> 18p
- R25, R26: value 22R -> 27R
Connections:
- net SR_CLK is gone; now on net USBC_DAM: U3.37 (GPIO25)
- net SR_nEN is gone; now on net SD_DET: U3.31 (GPIO20)
- net SW4 is gone; now on net AIN1: U3.39 (GPIO27_ADC1)
- net +3V3: now also C10.1, C9.1, U2.8 (VCC), C45.1, U11.1 (IN), U8.5 (VCC)
- net +5V: now also U7.8 (Vcc); no longer C10.1, C9.1, U2.8 (VCC)
- net AIN1: no longer U3.41 (GPIO29_ADC3)
- net CC1_DET: now also U7.1, U8.1
- net CC2_DET: now also U7.7, U8.2
- net GND: now also C45.2, C46.2, U11.3 (GND), U7.4 (Vee), U8.3 (GND)
- net SD_DET: no longer U3.18 (GPIO15)
- net UC_CC1: now also U7.3 (+)
- net UC_CC2: now also U7.5 (+)
- net USBC_CC_THRES: now also U7.2 (-), U7.6 (-)
- net USBC_DAM: now also U8.4
- net AIN0 renamed AIN2
- net Audio_EN renamed I2C1_SDA
- net PWM renamed SWI3
- net SR_DAT renamed WS2812_LV
- net SR_LATCH renamed SWI4
- net SW1 renamed SWI1
- net SW2 renamed SWI2
- net SW3 renamed 2v048_REF
- net 2v048_REF: now also C46.1, U11.2 (OUT)
- new net AIN3: U3.41 (GPIO29_ADC3)
- new net I2C1_SCL: U3.18 (GPIO15)
Other:
- moved on the sheet: R10, R9

Commit message: Update PCB
Connections:
- net SD_DET: now also U3.2 (GPIO0); no longer U3.31 (GPIO20)
- net SPI0_MISO: now also U3.31 (GPIO20); no longer U3.2 (GPIO0)
- net SWI1: now also U3.4 (GPIO2); no longer U3.29 (GPIO18)
- net SWI2: now also U3.5 (GPIO3); no longer U3.30 (GPIO19)
- net SWI3: now also U3.6 (GPIO4); no longer U3.34 (GPIO22)
- net at R2.1: now also U3.29 (GPIO18); no longer U3.4 (GPIO2)
- net at R3.1: now also U3.30 (GPIO19); no longer U3.5 (GPIO3)
- net at R1.1: now also U3.34 (GPIO22); no longer U3.6 (GPIO4)
Other:
- note added: "Bottom"
- note added: "RHS"
- note added: "Top"

Commit message: Finish layout
Connections:
- net +3V3: now also R22.1
- net +5V: no longer R22.1
- net USB_SHLD: now reaches C8.1, J3.S1 (SHIELD), R11.1
Changed lines of the file:
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@@
 		)
 	)
+	(label "USB_SHLD"
+		(at 25.4 118.11 0)
+		(fields_autoplaced yes)
+		(effects
+			(font
+				(size 1.27 1.27)
+			)
+			(justify left bottom)
+		)
+	)
 	(label "SWCLK"
 		(at 171.45 154.94 0)
@@
 	)
 	(symbol
-		(lib_id "power:+5V")
-		(at 21.59 167.64 0)
-		(unit 1)
-		(exclude_from_sim no)
-		(in_bom yes)
-		(on_board yes)
-		(dnp no)
-		(fields_autoplaced yes)
-		(property "Reference" "#PWR081"
-			(at 21.59 171.45 0)
-			(effects
-				(font
-					(size 1.27 1.27)
-				)
-				(hide yes)
-			)
-		)
-		(property "Value" "+5V"
-			(at 21.59 162.56 0)
-			(effects
-				(font
-					(size 1.27 1.27)
-				)
-			)
-		)
-		(property "Footprint" ""
-			(at 21.59 167.64 0)
-			(effects
-				(font
-					(size 1.27 1.27)
-				)
-				(hide yes)
-			)
-		)
-		(property "Datasheet" ""
-			(at 21.59 167.64 0)
-			(effects
-				(font
-					(size 1.27 1.27)
-				)
-				(hide yes)
-			)
-		)
-		(property "Description" "Power symbol creates a global label with name \"+5V\""
-			(at 21.59 167.64 0)
-			(effects
-				(font
-					(size 1.27 1.27)
-				)
-				(hide yes)
-			)
-		)
-		(pin "1"
-		)
-		(instances
-			(project "better-lamp-controller"
-				(path "/714ed833-23d9-46bd-9c89-d82c98fb7d43/b624bc1a-d25e-4c09-9e43-4b433f036622"
-					(reference "#PWR081")
-					(unit 1)
-				)
-			)
-		)
-	)
-	(symbol
 		(lib_id "Device:R")
 		(at 34.29 121.92 0)
@@
 					(unit 1)
 				)
+			)
+		)
+	)
+	(symbol
+		(lib_id "power:+3V3")
+		(at 21.59 167.64 0)
+		(unit 1)
+		(exclude_from_sim no)
+		(in_bom yes)
+		(on_board yes)
+		(dnp no)
+		(fields_autoplaced yes)
+		(property "Reference" "#PWR018"
+			(at 21.59 171.45 0)
+			(effects
+				(font
+					(size 1.27 1.27)
+				)
+				(hide yes)
+			)
+		)
+		(property "Value" "+3V3"
+			(at 21.59 162.56 0)
+			(effects
+				(font
+					(size 1.27 1.27)
+				)
+			)
+		)
+		(property "Footprint" ""
+			(at 21.59 167.64 0)
+			(effects
+				(font
+					(size 1.27 1.27)
+				)
+				(hide yes)
+			)
+		)
+		(property "Datasheet" ""
+			(at 21.59 167.64 0)
+			(effects
+				(font
+					(size 1.27 1.27)
+				)
+				(hide yes)
+			)
+		)
+		(property "Description" "Power symbol creates a global label with name \"+3V3\""
+			(at 21.59 167.64 0)
+			(effects
+				(font
+					(size 1.27 1.27)
+				)
+				(hide yes)
+			)
+		)
+		(pin "1"
+		)
+		(instances
+			(project "better-lamp-controller"
+				(path "/714ed833-23d9-46bd-9c89-d82c98fb7d43/b624bc1a-d25e-4c09-9e43-4b433f036622"
+					(reference "#PWR018")
+					(unit 1)
+				)
