File: better-lamp-controller.kicad_pcb (KiCad board)
At the start: 2 copper layers, 89 parts, among them J1 Conn_02x20_Odd_Even, J2 Micro_SD_Card_Det_Hirose_DM3AT, J3 HC-TYPE-C-16P-01A, J4 Conn_02x10_Odd_Even, J5 Conn_01x05_Pin, J6 Conn_01x02_Pin, J7 Conn_01x04_Pin, J8 Conn_01x04_Pin, J9 Conn_ARM_JTAG_SWD_10, U1 LP5860T, U2 74LVC2G66, U3 RP2040, U4 MAX98360A, U5 W25Q16JVSS, U6 74AHCT1G08, U7 LM393PWR, U8 74AHCT1G08, U9 LMR33620BDDA, Y1 RH100-12.000-18-2030-TR

Commit message: Add stackup
Parts:
- removed C36: 0u1, Capacitor_SMD:C_0603_1608Metric_Pad1.08x0.95mm_HandSolder
- added C43: 0u1, Capacitor_SMD:C_0603_1608Metric_Pad1.08x0.95mm_HandSolder, F.Cu at (50.9, -31.8)
- added R23: 10k, Resistor_SMD:R_0603_1608Metric_Pad0.98x0.95mm_HandSolder, F.Cu at (50.9, -24.3)
- added U10: PCF2131, kicad global library:HLSON16_SOT1992-1, F.Cu at (7.73, -18.5)
- moved C11 71.8 mm to (50.9, -36.8)
- moved C12 71.8 mm to (50.9, -34.3)
- moved R15 53.7 mm to (50.9, -26.8)
- moved R12 50.6 mm to (50.9, -29.3)
- moved J2 42.3 mm to (40.3, -28.7)
Connections:
- net /MCU/SD_SPI_CS renamed /SPI1_SD_CS
- net /MCU/SD_SPI_MISO renamed /SPI1_MISO
- net /MCU/SD_SPI_MOSI renamed /SPI1_MOSI
- net /MCU/SD_SPI_SCK renamed /SPI1_SCK
- C12 pad 1: +3V3 -> /SD_DET
- J1 pad 39: /Ext_CS2 -> /Ext_CS1
- J1 pad 40: /Ext_CS3 -> /Ext_CS2
- J2 pad 10: unconnected-(J2-DET_A-Pad10) -> /SD_DET
- J2 pad 9: unconnected-(J2-DET_B-Pad9) -> GND
- J3 pad A8: /MCU/SWCLK_GATED -> /MCU/SWD_GATED
- J3 pad B8: /MCU/SWD_GATED -> /MCU/SWCLK_GATED
- J4 pad 10: /SW0 -> +5V
- R6 pad 2: /MCU/I2S_LRCLK -> /LRCLK
- R7 pad 2: /MCU/I2S_BCLK -> /BCLK
- R8 pad 2: /MCU/I2S_DAT -> /AUDIO_DAT
- U3 pad 12: /Ext_CS1 -> /SPI1_RTC_CS
- U3 pad 13: /MCU/Audio_EN -> /Audio_EN
- U3 pad 18: /MCU/SD_DET -> /SD_DET
- U3 pad 27: /SW0 -> /RTC_INT
- U3 pad 28: /Ext_CS2 -> /Ext_CS1
- U3 pad 31: /MCU/SR_nEN -> /nEN
- U3 pad 32: /Ext_CS3 -> /Ext_CS2
- U3 pad 34: /MCU/PWM -> /PWM
- U3 pad 35: /MCU/SR_LATCH -> /LATCH
- U3 pad 36: /MCU/SR_DAT -> /DAT
- U3 pad 37: /MCU/SR_CLK -> /CLK
Other:
- copper layers 2 -> 4

Commit message: Begin layout
Parts:
- removed C25: 0u1, Capacitor_SMD:C_0603_1608Metric_Pad1.08x0.95mm_HandSolder
- added BT1: CR2032 Lithium Primary, Battery:BatteryHolder_Keystone_3000_1x12mm, F.Cu at (96.2, 127.7)
- added C36: 1u, Capacitor_SMD:C_0805_2012Metric_Pad1.18x1.45mm_HandSolder, F.Cu at (102.0, 110.8)
- added C44: 0u1, Capacitor_SMD:C_0603_1608Metric_Pad1.08x0.95mm_HandSolder, F.Cu at (99.2, 107.9)
- added R24: 470R, Resistor_SMD:R_0603_1608Metric_Pad0.98x0.95mm_HandSolder, F.Cu at (101.9, 112.5)
- added R25: 22R, Resistor_SMD:R_0603_1608Metric_Pad0.98x0.95mm_HandSolder, F.Cu at (120.2, 88.8)
- added R26: 22R, Resistor_SMD:R_0603_1608Metric_Pad0.98x0.95mm_HandSolder, F.Cu at (121.7, 88.8)
- JP1: moved to B.Cu
- moved J1 229.6 mm to (157.9, 129.6), turned to 180 degrees
- moved J5 211.5 mm to (178.0, 124.6)
- moved J4 206.9 mm to (142.8, 129.0), turned to -90 degrees
- moved JP2 206.3 mm to (195.9, 50.9)
- moved JP3 206.3 mm to (195.9, 54.5)
- moved JP4 206.3 mm to (195.9, 58.0)
- moved JP5 206.3 mm to (195.9, 61.5)
- moved J8 184.9 mm to (159.3, 67.0), turned to 90 degrees
- moved C29 181.7 mm to (143.0, 116.9)
- moved U1 179.4 mm to (145.9, 100.0)
- moved C4 175.8 mm to (146.1, 105.6), turned to -90 degrees
- moved J6 175.1 mm to (110.7, 129.0)
- moved C1 175.0 mm to (148.9, 95.0)
- moved C3 174.4 mm to (144.0, 94.0), turned to 90 degrees
- moved R4 172.8 mm to (145.5, 94.0), turned to 90 degrees
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Connections:
- J9 pad 2: /MCU/SWDIO -> /MCU/SWD
- R23 pad 2: Net-(U10-nINTA) -> /RTC_INT
- U10 pad 13: Net-(U10-nINTA) -> /RTC_INT
- U10 pad 15: +3V3 -> /RTC_Vdd
- U10 pad 16: unconnected-(U10-Vbat-Pad16) -> /RTC_VBat
- U3 pad 46: /MCU/USB_D- -> Net-(U3-USB_DM)
- U3 pad 47: /MCU/USB_D+ -> Net-(U3-USB_DP)
Other:
- board outline added: 100 x 99.9 mm

Commit message: Update layout
Parts:
- removed J8: Conn_01x04_Pin, Connector_PinHeader_2.54mm:PinHeader_1x04_P2.54mm_Vertical
- removed R18, R19: 10k, Resistor_SMD:R_0603_1608Metric_Pad0.98x0.95mm_HandSolder
- added C25: 0u1, Capacitor_SMD:C_0603_1608Metric_Pad1.08x0.95mm_HandSolder, F.Cu at (120.6, 91.1)
- added C45: 0u1, Capacitor_SMD:C_0603_1608Metric_Pad1.08x0.95mm_HandSolder, F.Cu at (124.0, 85.6)
- added C46: 1u, Capacitor_SMD:C_0805_2012Metric_Pad1.18x1.45mm_HandSolder, F.Cu at (124.3, 90.8)
- added C47: 0u1, Capacitor_SMD:C_0603_1608Metric_Pad1.08x0.95mm_HandSolder, F.Cu at (137.2, 118.4)
- added H1: MountingHole_Pad, MountingHole:MountingHole_3.2mm_M3_Pad, F.Cu at (150.0, 76.0)
- added H2: MountingHole_Pad, MountingHole:MountingHole_3.2mm_M3_Pad, F.Cu at (150.0, 127.0)
- added H3: MountingHole_Pad, MountingHole:MountingHole_3.2mm_M3_Pad, F.Cu at (80.0, 127.0)
- added H4: MountingHole_Pad, MountingHole:MountingHole_3.2mm_M3_Pad, F.Cu at (80.0, 76.0)
- added R27: 1k3, Resistor_SMD:R_0603_1608Metric_Pad0.98x0.95mm_HandSolder, F.Cu at (119.1, 115.0)
- added R28: 1k3, Resistor_SMD:R_0603_1608Metric_Pad0.98x0.95mm_HandSolder, F.Cu at (119.1, 116.5)
- added U11: MAX6106, Package_TO_SOT_SMD:SOT-23, F.Cu at (124.3, 88.0)
- added U12: OPT4048, kicad global library:SOT-583_DTS, F.Cu at (137.2, 114.8)
- C27, C28: value 27p -> 18p
- JP2, JP3, JP4, JP5: moved to B.Cu
- R25, R26: value 22R -> 27R
- U6, U8: value 74AHCT1G08 -> 74LVC1G08
- U7: value LM393PWR -> TLV7012; footprint Package_SO:TSSOP-8_4.4x3mm_P0.65mm -> Package_TO_SOT_SMD:TSOT-23-8
- moved J5 59.8 mm to (141.5, 77.3)
- moved JP2 54.0 mm to (155.0, 86.1)
- moved R11 52.8 mm to (78.4, 81.2), turned to 180 degrees
- moved JP3 50.3 mm to (155.0, 83.6)
- moved JP5 49.1 mm to (155.0, 88.6)
- moved J3 48.1 mm to (79.2, 87.3), turned to -90 degrees
- moved C8 48.1 mm to (81.7, 81.2), turned to 0 degrees
- moved JP4 47.0 mm to (155.0, 81.0)
- moved U9 41.9 mm to (110.5, 80.1), turned to 180 degrees
- moved L1 41.8 mm to (110.3, 85.3)
- moved C33 41.5 mm to (115.8, 83.5), turned to 90 degrees
- moved C14 40.2 mm to (117.5, 77.8)
- moved R10 38.2 mm to (86.0, 90.7), turned to 0 degrees
- moved C34 37.7 mm to (119.2, 83.5), turned to 90 degrees
- moved R9 37.6 mm to (87.2, 81.5), turned to 90 degrees
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Connections:
- net Net-(U9-SW) renamed /3v3 Regulator/REG_SW
- C10 pad 1: +5V -> +3V3
- C37 pad 1: /SW1 -> /SWI1
- C38 pad 1: /SW2 -> /SWI2
- C39 pad 1: /SW3 -> /SWI3
- C40 pad 1: /SW4 -> /SWI4
- C41 pad 2: /AIN1 -> /AIN2
- C42 pad 2: /AIN0 -> /AIN1
- C9 pad 1: +5V -> +3V3
- J1 pad 1: /SW0 -> /CS1
- J1 pad 10: /SW9 -> /CS8
- J1 pad 11: /SW10 -> /SW3
- J1 pad 12: /CS1 -> /SW0
- J1 pad 13: /CS0 -> /SW5
- J1 pad 14: /CS3 -> /SW2
- J1 pad 15: /CS2 -> /SW7
- J1 pad 16: /CS5 -> /SW4
- J1 pad 17: /CS4 -> /SW9
- J1 pad 18: /CS7 -> /SW6
- J1 pad 19: /CS6 -> /SW8
- J1 pad 2: /SW1 -> /CS0
- J1 pad 20: /CS9 -> unconnected-(J1-Pin_20-Pad20)
- J1 pad 21: /CS8 -> /SW10
- J1 pad 22: /CS11 -> /CS9
- J1 pad 24: /CS13 -> /CS11
- J1 pad 26: /CS15 -> /CS13
- J1 pad 28: /CS17 -> /CS15
- J1 pad 3: /SW2 -> /CS3
- J1 pad 30: /EXT_VSYNC -> /CS17
- J1 pad 35: +3V3 -> /EXT_VSYNC
- J1 pad 4: /SW3 -> /CS2
- J1 pad 5: /SW4 -> /CS5
- J1 pad 6: /SW5 -> /CS4
- J1 pad 7: /SW6 -> /CS7
- J1 pad 8: /SW7 -> /CS6
- J1 pad 9: /SW8 -> /SW1
- J4 pad 1: /DAT -> /I2C_SCL
- J4 pad 10: +5V -> GND
- J4 pad 11: /SW1 -> /SWI1
- J4 pad 12: /SW2 -> /SWI2
- J4 pad 13: /SW3 -> /SWI3
- J4 pad 14: /SW4 -> /SWI4
- J4 pad 15: GND -> /Vref
- J4 pad 16: /AIN0 -> /AIN1
- J4 pad 17: GND -> /AIN3
- J4 pad 18: /AIN1 -> /AIN2
- J4 pad 2: /LATCH -> GND
- J4 pad 3: /CLK -> /I2C_SDA
- J4 pad 4: /PWM -> unconnected-(J4-Pin_4-Pad4)
- J4 pad 5: /nEN -> GND
- J4 pad 6: GND -> +5V
- U2 pad 8: +5V -> +3V3
- U3 pad 13: /Audio_EN -> /I2C_SDA
- U3 pad 18: /SD_DET -> /I2C_SCL
- U3 pad 29: /SW1 -> /SWI1
- U3 pad 30: /SW2 -> /SWI2
- U3 pad 31: /nEN -> /SD_DET
- U3 pad 34: /PWM -> /SWI3
- U3 pad 35: /LATCH -> /SWI4
- U3 pad 36: /DAT -> /WS2812_LV
- U3 pad 37: /CLK -> /MCU/USBC_DAM
- U3 pad 38: /SW3 -> /Vref
- U3 pad 39: /SW4 -> /AIN1
- U3 pad 40: /AIN0 -> /AIN2
- U3 pad 41: /AIN1 -> /AIN3
- U4 pad 6: /Audio_EN -> +5V
- U8 pad 5: +5V -> +3V3
Routing:
- net /SPI1_SD_CS: track 0.00 -> 36.4 mm, vias 0 -> 2
- net +3V3: track 0.00 -> 30.9 mm
- net /CS16: track 0.00 -> 23.1 mm
- net /CS17: track 0.00 -> 21.5 mm
- net /CS14: track 0.00 -> 20.6 mm
- net /CS7: track 0.00 -> 18.9 mm
- net /CS15: track 0.00 -> 18.8 mm
- net /CS12: track 0.00 -> 17.6 mm
- net /SW1: track 0.00 -> 16.9 mm
- net /CS13: track 0.00 -> 16.3 mm
- net /SW7: track 0.00 -> 15.4 mm
- net /CS10: track 0.00 -> 15.3 mm
- net /SW3: track 0.00 -> 15.0 mm, vias 0 -> 1
- net /CS8: track 0.00 -> 14.6 mm
- net /SW9: track 0.00 -> 14.3 mm
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- added copper zone on F.Cu, net +3V3
- added copper zone on F.Cu, net +5V
Other:
- board size 100 x 99.9 mm -> 90 x 60 mm

Commit message: Update PCB
Parts:
- moved C25 29.0 mm to (117.0, 119.9), turned to 0 degrees
- moved C42 28.8 mm to (120.4, 119.9), turned to 0 degrees
- moved C41 27.4 mm to (120.4, 118.4), turned to 180 degrees
- moved R28 22.1 mm to (141.0, 119.6), turned to 180 degrees
- moved R27 18.2 mm to (136.7, 119.6)
- moved JP4 18.1 mm to (140.7, 92.0)
- moved JP2 18.0 mm to (140.7, 97.0)
- moved JP3 18.0 mm to (140.7, 94.5)
- moved JP5 18.0 mm to (140.7, 99.5)
- moved R2 16.5 mm to (127.2, 95.0), turned to 90 degrees
- moved R1 15.6 mm to (121.7, 93.5), turned to 90 degrees
- moved R3 15.2 mm to (125.7, 95.0), turned to 90 degrees
- moved C7 8.88 mm to (105.5, 118.8), turned to -90 degrees
- moved C47 5.53 mm to (132.9, 115.0), turned to 90 degrees
- moved U4 4.38 mm to (111.6, 117.3), turned to -90 degrees
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Connections:
- R1 pad 1: Net-(U3-GPIO4) -> Net-(U3-GPIO22)
- R2 pad 1: Net-(U3-GPIO2) -> Net-(U3-GPIO18)
- R3 pad 1: Net-(U3-GPIO3) -> Net-(U3-GPIO19)
- U3 pad 2: /LED_MISO -> /SD_DET
- U3 pad 29: /SWI1 -> Net-(U3-GPIO18)
- U3 pad 30: /SWI2 -> Net-(U3-GPIO19)
- U3 pad 31: /SD_DET -> /LED_MISO
- U3 pad 34: /SWI3 -> Net-(U3-GPIO22)
- U3 pad 4: Net-(U3-GPIO2) -> /SWI1
- U3 pad 5: Net-(U3-GPIO3) -> /SWI2
- U3 pad 6: Net-(U3-GPIO4) -> /SWI3
Routing:
- net /Ext_CS0: track 2.63 -> 58.3 mm, vias 1 -> 2
- net /Vref: track 0.00 -> 54.0 mm, vias 0 -> 1
- net /AIN1: track 0.00 -> 52.7 mm, vias 0 -> 2
- net /SWI4: track 0.00 -> 52.0 mm, vias 0 -> 2
- net /AIN2: track 0.00 -> 49.6 mm, vias 0 -> 2
- net /Ext_CS1: track 0.00 -> 47.9 mm, vias 0 -> 2
- net /Ext_CS2: track 0.00 -> 47.1 mm, vias 0 -> 2
- net /SPI1_SCK: track 0.00 -> 46.5 mm, vias 0 -> 2
- net /AIN3: track 0.00 -> 46.0 mm, vias 0 -> 2
- net /SPI1_MOSI: track 0.00 -> 42.8 mm, vias 0 -> 4
- net /SPI1_MISO: track 0.00 -> 40.6 mm, vias 0 -> 5
- net /MCU/USB_D-: track 0.00 -> 40.5 mm
- net /MCU/USB_D+: track 0.00 -> 40.5 mm
- net GND: track 0.00 -> 33.6 mm, vias 0 -> 19
- net /LED_MISO: track 0.00 -> 33.3 mm, vias 0 -> 3
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
Commit message: Finish layout
Parts:
- removed C11: 1n, Capacitor_SMD:C_0603_1608Metric_Pad1.08x0.95mm_HandSolder
- removed R12: 100k, Resistor_SMD:R_0603_1608Metric_Pad0.98x0.95mm_HandSolder
- moved C10 4.21 mm to (101.0, 81.7), turned to -90 degrees
- moved C13 3.24 mm to (83.5, 114.7), turned to 0 degrees
- moved C31 1.16 mm to (104.1, 78.4)
- moved C30 0.99 mm to (115.2, 79.8)
- moved C34 0.99 mm to (118.5, 82.8)
- moved R20 0.99 mm to (105.5, 76.0)
- moved R21 0.99 mm to (108.8, 76.0)
- moved U9 0.99 mm to (109.8, 79.4)
- moved C14 0.99 mm to (116.8, 77.1)
- moved C33 0.99 mm to (115.2, 82.8)
- moved L1 0.99 mm to (109.6, 84.7)
- moved C32 0.98 mm to (105.2, 81.3)
- moved C18 0.85 mm to (117.6, 107.4)
- moved C29 0.36 mm to (134.5, 83.3), turned to -90 degrees
Connections:
- net Net-(J3-SHIELD) renamed /MCU/USB_SHLD
- J2 pad 11: Net-(J2-SHIELD) -> GND
- R22 pad 1: +5V -> +3V3
Routing:
- net GND: track 33.6 -> 92.5 mm, vias 19 -> 155
- net /SD_DET: track 4.88 -> 54.3 mm, vias 0 -> 2
- net +3V3: track 43.1 -> 89.3 mm, vias 3 -> 26
- net /MCU/SWCLK: track 24.8 -> 66.7 mm, vias 1 -> 3
- net /RTC_INT: track 6.19 -> 46.8 mm, vias 1 -> 2
- net /MCU/SWD: track 19.1 -> 58.3 mm, vias 1 -> 3
- net /SPI1_RTC_CS: track 1.96 -> 30.0 mm, vias 1 -> 4
- net /MCU/USBC_DAM: track 21.9 -> 48.4 mm
- net /WS2812_LV: track 0.00 -> 24.9 mm, vias 0 -> 2
- net +1V1: track 14.1 -> 38.4 mm, vias 1 -> 3
- net /I2C_SCL: track 13.1 -> 31.6 mm, vias 1 -> 0
- net /I2C_SDA: track 11.6 -> 29.6 mm
- net /MCU/UC_CC2: track 3.75 -> 19.0 mm, vias 0 -> 2
- net +5V: track 17.0 -> 28.6 mm, vias 7 -> 17
- net /MCU/UC_CC1: track 3.47 -> 13.5 mm
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- added copper zone on In2.Cu, net +3V3
- added copper zone on In2.Cu, net +5V
- added copper zone on F.Cu, net /3v3 Regulator/REG_SW
- added copper zone on F.Cu, net /MCU/USB_SHLD
- added copper zone on B.Cu, net GND
- added copper zone on F.Cu, net GND
- added copper zone on In1.Cu, net GND

Commit message: Update IO Board
Parts:
- moved C45 0.30 mm to (124.0, 85.3)
Routing:
- net +3V3: track 89.3 -> 90.7 mm, vias 26 -> 27
- net GND: track 92.5 -> 93.2 mm, vias 155 -> 333

Commit message: Update IO board
Connections:
- J4 pad 4: unconnected-(J4-Pin_4-Pad4) -> GND
