File: better-lamp-controller.kicad_sch (KiCad schematic)
At the start: 23 parts, among them J1 Conn_02x20_Odd_Even, J4 Conn_02x10_Odd_Even, J5 Conn_01x05_Pin, J6 Conn_01x02_Pin, J7 Conn_01x04_Pin, J8 Conn_01x04_Pin, U1 LP5860T, U2 DRV8837C, U4 MAX98360A, U6 74AHCT1G08

Commit message: Add RTC
Parts:
- removed C2: 0u1, symbol Device:C
- removed U2: DRV8837C, Package_SON:WSON-8-1EP_2x2mm_P0.5mm_EP0.9x1.6mm, symbol Driver_Motor:DRV8837C
- added C11: 1n, Capacitor_SMD:C_0603_1608Metric_Pad1.08x0.95mm_HandSolder, symbol Device:C
- added C12, C37, C38, C39, C40, C41, C42, C43: 0u1, Capacitor_SMD:C_0603_1608Metric_Pad1.08x0.95mm_HandSolder, symbol Device:C
- added C13: 100u, Capacitor_THT:CP_Radial_D10.0mm_P5.00mm, symbol Device:C_Polarized
- added J2: Micro_SD_Card_Det_Hirose_DM3AT, Connector_Card:microSD_HC_Hirose_DM3AT-SF-PEJM5, symbol Connector:Micro_SD_Card_Det_Hirose_DM3AT
- added R12: 100k, Resistor_SMD:R_0603_1608Metric_Pad0.98x0.95mm_HandSolder, symbol Device:R
- added R15: 43R, Resistor_SMD:R_0603_1608Metric_Pad0.98x0.95mm_HandSolder, symbol Device:R
- added R23: 10k, Resistor_SMD:R_0603_1608Metric_Pad0.98x0.95mm_HandSolder, symbol Device:R
- added U10: PCF2131, kicad global library:HLSON16_SOT1992-1, symbol Global:PCF2131
- C1: value 0u1 -> 1u; footprint (none) -> Capacitor_SMD:C_0805_2012Metric_Pad1.18x1.45mm_HandSolder
- C29, C3, C6: footprint (none) -> Capacitor_SMD:C_0603_1608Metric_Pad1.08x0.95mm_HandSolder
- C4, C5: footprint (none) -> Capacitor_SMD:C_0805_2012Metric_Pad1.18x1.45mm_HandSolder
- C7: footprint (none) -> Capacitor_SMD:C_1210_3225Metric
- J1: footprint (none) -> Connector_IDC:IDC-Header_2x20_P2.54mm_Vertical
- J4: footprint (none) -> Connector_IDC:IDC-Header_2x10_P2.54mm_Vertical
- J5: footprint (none) -> Connector_PinHeader_2.54mm:PinHeader_1x05_P2.54mm_Vertical
- J6: footprint (none) -> Connector_PinHeader_2.54mm:PinHeader_1x02_P2.54mm_Vertical
- J7, J8: footprint (none) -> Connector_PinHeader_2.54mm:PinHeader_1x04_P2.54mm_Vertical
- JP2, JP3, JP4, JP5: footprint (none) -> Jumper:SolderJumper-2_P1.3mm_Open_RoundedPad1.0x1.5mm
- R4: footprint (none) -> Resistor_SMD:R_0603_1608Metric_Pad0.98x0.95mm_HandSolder
- U6: footprint (none) -> Package_TO_SOT_SMD:SOT-23-5
Connections:
- net +VSW is gone; now on net +5V: J4.7 (Pin_7)
- net VFb is gone; now on net GND: J4.6 (Pin_6)
- net +3V3: now also J4.9 (Pin_9), C43.1, J2.4 (VDD), R23.1, U10.15 (Vdd); no longer C1.1, J4.10 (Pin_10)
- net +5V: now also J4.10 (Pin_10), C13.1
- net AIN0: now also J4.16 (Pin_16), C42.2; no longer J4.18 (Pin_18)
- net AIN1: now also J4.18 (Pin_18), C41.2; no longer J4.20 (Pin_20)
- net Audio+: now also J4.19 (Pin_19)
- net Audio-: now also J4.20 (Pin_20)
- net Ext_CS1: now also J1.39 (Pin_39); no longer J1.40 (Pin_40)
- net GND: now also J4.15 (Pin_15), C11.2, C12.2, C13.2, C37.2, C38.2, C39.2, C40.2, C41.1, C42.1, C43.2, J2.6 (VSS), J2.9 (DET_B), R12.2, U10.1 (IFS), U10.17 (EP), U10.7 (Vss); no longer J1.39 (Pin_39), J4.19 (Pin_19), J4.9 (Pin_9)
- net SW1: now also C37.1
- net SW2: now also C38.1
- net SW3: now also C39.1
- net SW4: now also C40.1
- net SW5: no longer J4.15 (Pin_15)
- net SW6: no longer J4.16 (Pin_16)
- net at U1.32 (VCAP): now also C1.1
- net VFa renamed nEN
- new net: C11.1, J2.11 (SHIELD), R12.1
- new net: J2.7 (DAT0), R15.1
- new net: R23.2, U10.13 (nINTA)
- new net Ext_CS2: J1.40 (Pin_40)
- new net SD_DET: C12.1, J2.10 (DET_A)
- new net SPI1_MISO: R15.2, U10.4 (SDO)
- new net SPI1_MOSI: J2.3 (CMD), U10.3 (SDI)
- new net SPI1_RTC_CS: U10.5 (SDA/nCE)
- new net SPI1_SCK: J2.5 (CLK), U10.2 (SCL)
- new net SPI1_SD_CS: J2.2 (DAT3/CD)
- no-connect marks 0 -> 7
Other:
- removed sheet 3v3 LDO
- removed sheet VFD Power
- added sheet 3v3 Regulator (Step Down.kicad_sch)
- sheet MCU ports: added AIN0, AIN1, PWM, RTC_INT, SD_DET, SPI0_EXT_CS2, SPI1_MISO, SPI1_MOSI, SPI1_RTC_CS, SPI1_SCK, SPI1_SD_CS, SR_CLK, SR_DAT, SR_LATCH, SR_nEN, SW1, SW2, SW3, SW4; removed none
- moved on the sheet: C29, C3, C4, C5, C6, C7, J1, J4, J5, J6, J7, J8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

Commit message: Begin layout
Parts:
- added BT1: CR2032 Lithium Primary, Battery:BatteryHolder_Keystone_3000_1x12mm, symbol Device:Battery_Cell
- added C36: 1u, Capacitor_SMD:C_0805_2012Metric_Pad1.18x1.45mm_HandSolder, symbol Device:C
- added C44: 0u1, Capacitor_SMD:C_0603_1608Metric_Pad1.08x0.95mm_HandSolder, symbol Device:C
- added R24: 470R, Resistor_SMD:R_0603_1608Metric_Pad0.98x0.95mm_HandSolder, symbol Device:R
Connections:
- net +3V3: now also R24.1; no longer U10.15 (Vdd)
- net GND: now also BT1.2 (-), C36.2, C44.2
- net RTC_INT: now also R23.2, U10.13 (nINTA)
- net RTC_VBat: now reaches U10.16 (Vbat)
- net RTC_VBat: now also BT1.1 (+), C44.1
- new net RTC_Vdd: C36.1, R24.2, U10.15 (Vdd)
- no-connect marks 7 -> 9
Other:
- moved on the sheet: R23

Commit message: Update layout
Parts:
- removed J8: Conn_01x04_Pin, Connector_PinHeader_2.54mm:PinHeader_1x04_P2.54mm_Vertical, symbol Connector:Conn_01x04_Pin
- removed U6: 74AHCT1G08, Package_TO_SOT_SMD:SOT-23-5, symbol 74xGxx:74AHCT1G08
- added C25, C47: 0u1, Capacitor_SMD:C_0603_1608Metric_Pad1.08x0.95mm_HandSolder, symbol Device:C
- added H1, H2, H3, H4: MountingHole_Pad, MountingHole:MountingHole_3.2mm_M3_Pad, symbol Mechanical:MountingHole_Pad
- added R27, R28: 1k3, Resistor_SMD:R_0603_1608Metric_Pad0.98x0.95mm_HandSolder, symbol Device:R
- added U12: OPT4048, kicad global library:SOT-583_DTS, symbol Global:OPT4048
- added U6: 74LVC1G08, Package_TO_SOT_SMD:SOT-23-5, symbol Global:SN74LV1T08
Connections:
- net AIN0 is gone; now on net AIN1: C42.2, J4.16 (Pin_16)
- net Audio_EN is gone; now on net +5V: U4.6 (EN)
- net LATCH is gone; now on net GND: J4.2 (Pin_2)
- net nEN is gone; now on net GND: J4.5 (Pin_5)
- net +3V3: now also C47.1, R27.1, R28.1, U12.1 (Vdd); no longer J1.35 (Pin_35)
- net +5V: now also J4.6 (Pin_6), U6.1, U6.5 (VCC); no longer J4.10 (Pin_10)
- net AIN1: no longer C41.2, J4.18 (Pin_18)
- net CS0: now also J1.2 (Pin_2); no longer J1.13 (Pin_13)
- net CS1: now also J1.1 (Pin_1); no longer J1.12 (Pin_12)
- net CS11: now also J1.24 (Pin_24); no longer J1.22 (Pin_22)
- net CS13: now also J1.26 (Pin_26); no longer J1.24 (Pin_24)
- net CS15: now also J1.28 (Pin_28); no longer J1.26 (Pin_26)
- net CS17: now also J1.30 (Pin_30); no longer J1.28 (Pin_28)
- net CS2: now also J1.4 (Pin_4); no longer J1.15 (Pin_15)
- net CS3: now also J1.3 (Pin_3); no longer J1.14 (Pin_14)
- net CS4: now also J1.6 (Pin_6); no longer J1.17 (Pin_17)
- net CS5: now also J1.5 (Pin_5); no longer J1.16 (Pin_16)
- net CS6: now also J1.8 (Pin_8); no longer J1.19 (Pin_19)
- net CS7: now also J1.7 (Pin_7); no longer J1.18 (Pin_18)
- net CS8: now also J1.10 (Pin_10); no longer J1.21 (Pin_21)
- net CS9: now also J1.22 (Pin_22); no longer J1.20 (Pin_20)
- net EXT_VSYNC: now also J1.35 (Pin_35); no longer J1.30 (Pin_30)
- net GND: now also J4.10 (Pin_10), C25.1, C47.2, H1.1, H2.1, H3.1, H4.1, U12.2 (ADDR), U12.4 (GND), U6.3 (GND); no longer J4.15 (Pin_15), J4.17 (Pin_17), J4.6 (Pin_6)
- net SW0: now also J1.12 (Pin_12); no longer J1.1 (Pin_1)
- net SW1: now also J1.9 (Pin_9); no longer C37.1, J1.2 (Pin_2), J4.11 (Pin_11)
- net SW10: now also J1.21 (Pin_21); no longer J1.11 (Pin_11)
- net SW2: now also J1.14 (Pin_14); no longer C38.1, J1.3 (Pin_3), J4.12 (Pin_12)
- net SW3: now also J1.11 (Pin_11); no longer C39.1, J1.4 (Pin_4), J4.13 (Pin_13)
- net SW4: now also J1.16 (Pin_16); no longer C40.1, J1.5 (Pin_5), J4.14 (Pin_14)
- net SW5: now also J1.13 (Pin_13); no longer J1.6 (Pin_6)
- net SW6: now also J1.18 (Pin_18); no longer J1.7 (Pin_7)
- net SW7: now also J1.15 (Pin_15); no longer J1.8 (Pin_8)
- net SW8: now also J1.19 (Pin_19); no longer J1.9 (Pin_9)
- net SW9: now also J1.17 (Pin_17); no longer J1.10 (Pin_10)
- net WS2812_HV: now also U6.4
- net WS2812_LV: now also U6.2
- net CLK renamed I2C_SDA
- net I2C_SDA: now also R27.2, U12.8 (SDA)
- net DAT renamed I2C_SCL
- net I2C_SCL: now also R28.2, U12.5 (SCL)
- net PWM: no longer names the net of J4.4 (Pin_4)
- new net AIN2: C41.2, J4.18 (Pin_18)
- new net AIN3: C25.2, J4.17 (Pin_17)
- new net SWI1: C37.1, J4.11 (Pin_11)
- new net SWI2: C38.1, J4.12 (Pin_12)
- new net SWI3: C39.1, J4.13 (Pin_13)
- new net SWI4: C40.1, J4.14 (Pin_14)
- new net Vref: J4.15 (Pin_15)
- no-connect marks 9 -> 11
Other:
- sheet MCU ports: added 2v048_REF, AIN2, AIN3, I2C1_SCL, I2C1_SDA, SWI1, SWI2, SWI3, SWI4, WS2812_LV; removed AIN0, Audio_EN, PWM, SR_CLK, SR_DAT, SR_LATCH, SR_nEN, SW1, SW2, SW3, SW4
- note added: "Not using P20 to allow using IDE cables"
- moved on the sheet: BT1, C13, C29, C3, C36, C41, C42, C44, C6, C7, J7, R23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

Commit message: Finish layout
Parts:
- removed C11: 1n, Capacitor_SMD:C_0603_1608Metric_Pad1.08x0.95mm_HandSolder, symbol Device:C
- removed R12: 100k, Resistor_SMD:R_0603_1608Metric_Pad0.98x0.95mm_HandSolder, symbol Device:R
Connections:
- net GND: now also J2.11 (SHIELD)
Changed lines of the file:
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@@
 	)
 	(junction
-		(at 31.75 149.86)
-		(diameter 0)
-		(color 0 0 0 0)
-	)
-	(junction
 		(at 73.66 72.39)
 		(diameter 0)
@@
 	)
 	(junction
-		(at 31.75 142.24)
-		(diameter 0)
-		(color 0 0 0 0)
-	)
-	(junction
 		(at 285.75 198.12)
 		(diameter 0)
@@
 	(wire
 		(pts
-			(xy 27.94 142.24) (xy 31.75 142.24)
-		)
-		(stroke
-			(width 0)
-			(type default)
-		)
-	)
-	(wire
-		(pts
 			(xy 287.02 226.06) (xy 287.02 227.33)
 		)
@@
 	(wire
 		(pts
-			(xy 31.75 142.24) (xy 36.83 142.24)
+			(xy 200.66 85.09) (xy 196.85 85.09)
 		)
 		(stroke
@@
 	(wire
 		(pts
-			(xy 200.66 85.09) (xy 196.85 85.09)
+			(xy 127 184.15) (xy 127 172.72)
 		)
 		(stroke
@@
 	(wire
 		(pts
-			(xy 127 184.15) (xy 127 172.72)
+			(xy 31.75 137.16) (xy 31.75 149.86)
 		)
 		(stroke
@@
 	(wire
 		(pts
-			(xy 27.94 149.86) (xy 31.75 149.86)
-		)
-		(stroke
-			(width 0)
-			(type default)
-		)
-	)
-	(wire
-		(pts
 			(xy 62.23 48.26) (xy 62.23 55.88)
 		)
@@
 	(wire
 		(pts
-			(xy 31.75 137.16) (xy 31.75 142.24)
-		)
-		(stroke
-			(width 0)
-			(type default)
-		)
-	)
-	(wire
-		(pts
 			(xy 172.72 153.67) (xy 172.72 157.48)
 		)
@@
 	(wire
 		(pts
-			(xy 31.75 149.86) (xy 36.83 149.86)
-		)
-		(stroke
-			(width 0)
-			(type default)
-		)
-	)
-	(wire
-		(pts
 			(xy 85.09 127) (xy 74.93 127)
 		)
@@
 	)
 	(symbol
-		(lib_id "Device:C")
-		(at 27.94 146.05 0)
-		(unit 1)
-		(exclude_from_sim no)
-		(in_bom yes)
-		(on_board yes)
-		(dnp no)
-		(fields_autoplaced yes)
-		(property "Reference" "C11"
-			(at 31.75 144.7799 0)
-			(effects
-				(font
-					(size 1.27 1.27)
-				)
-				(justify left)
-			)
-		)
-		(property "Value" "1n"
-			(at 31.75 147.3199 0)
-			(effects
-				(font
-					(size 1.27 1.27)
-				)
-				(justify left)
-			)
-		)
-		(property "Footprint" "Capacitor_SMD:C_0603_1608Metric_Pad1.08x0.95mm_HandSolder"
-			(at 28.9052 149.86 0)
-			(effects
-				(font
-					(size 1.27 1.27)
-				)
-				(hide yes)
-			)
-		)
-		(property "Datasheet" "~"
-			(at 27.94 146.05 0)
-			(effects
-				(font
-					(size 1.27 1.27)
-				)
-				(hide yes)
-			)
-		)
-		(property "Description" "Unpolarized capacitor"
-			(at 27.94 146.05 0)
-			(effects
-				(font
-					(size 1.27 1.27)
-				)
-				(hide yes)
-			)
-		)
-		(pin "1"
-		)
-		(pin "2"
-		)
-		(instances
-			(project "better-lamp-controller"
-				(path "/714ed833-23d9-46bd-9c89-d82c98fb7d43"
-					(reference "C11")
-					(unit 1)
-				)
-			)
-		)
-	)
-	(symbol
 		(lib_id "Global:LP5860T")
 		(at 295.91 45.72 0)
@@
 					(unit 1)
 				)
-			)
-		)
-	)
-	(symbol
-		(lib_id "Device:R")
-		(at 36.83 146.05 0)
-		(unit 1)
-		(exclude_from_sim no)
-		(in_bom yes)
-		(on_board yes)
-		(dnp no)
-		(fields_autoplaced yes)
-		(property "Reference" "R12"
-			(at 39.37 144.7799 0)
-			(effects
-				(font
-					(size 1.27 1.27)
-				)
-				(justify left)
-			)
-		)
-		(property "Value" "100k"
-			(at 39.37 147.3199 0)
-			(effects
-				(font
-					(size 1.27 1.27)
-				)
-				(justify left)
-			)
-		)
-		(property "Footprint" "Resistor_SMD:R_0603_1608Metric_Pad0.98x0.95mm_HandSolder"
-			(at 35.052 146.05 90)
-			(effects
-				(font
-					(size 1.27 1.27)
-				)
-				(hide yes)
-			)
-		)
-		(property "Datasheet" "~"
-			(at 36.83 146.05 0)
-			(effects
-				(font
-					(size 1.27 1.27)
-				)
-				(hide yes)
-			)
-		)
-		(property "Description" "Resistor"
-			(at 36.83 146.05 0)
-			(effects
-				(font
-					(size 1.27 1.27)
-				)
-				(hide yes)
-			)
-		)
-		(pin "2"
-		)
-		(pin "1"
-		)
-		(instances
-			(project "better-lamp-controller"
-				(path "/714ed833-23d9-46bd-9c89-d82c98fb7d43"
-					(reference "R12")
-					(unit 1)
-				)

Commit message: Update IO board
Connections:
- net GND: now also J4.4 (Pin_4)
Changed lines of the file:
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@@
+	)
+	(symbol
+		(lib_id "power:GND")
+		(at 64.77 218.44 90)
+		(unit 1)
+		(exclude_from_sim no)
+		(in_bom yes)
+		(on_board yes)
+		(dnp no)
+		(property "Reference" "#PWR065"
+			(at 71.12 218.44 0)
+			(effects
+				(font
+					(size 1.27 1.27)
+				)
+				(hide yes)
+			)
+		)
+		(property "Value" "GND"
+			(at 67.564 218.44 90)
+			(effects
+				(font
+					(size 1.27 1.27)
+				)
+				(justify right)
+			)
+		)
+		(property "Footprint" ""
+			(at 64.77 218.44 0)
+			(effects
+				(font
+					(size 1.27 1.27)
+				)
+				(hide yes)
+			)
+		)
+		(property "Datasheet" ""
+			(at 64.77 218.44 0)
+			(effects
+				(font
+					(size 1.27 1.27)
+				)
+				(hide yes)
+			)
+		)
+		(property "Description" "Power symbol creates a global label with name \"GND\" , ground"
+			(at 64.77 218.44 0)
+			(effects
+				(font
+					(size 1.27 1.27)
+				)
+				(hide yes)
+			)
+		)
+		(pin "1"
+		)
+		(instances
+			(project "better-lamp-controller"
+				(path "/714ed833-23d9-46bd-9c89-d82c98fb7d43"
+					(reference "#PWR065")
+					(unit 1)
+				)
+			)
+		)
 	)
 	(symbol
