File: Alarm IO Board/buttons.kicad_sch (KiCad schematic)
At the start: 6 parts, among them SW1 SW_Push, SW2 SW_Push, SW3 SW_Push, SW4 SW_Push, SW5 SW_Push, SW6 SW_Push

Commit message: Update IO Board
Parts:
- SW1, SW2, SW3, SW4, SW5, SW6: value SW_Push -> Wurth WS-TATV; footprint (none) -> Button_Switch_THT:SW_PUSH_6mm
