File: Alarm IO Board/Alarm IO Board.kicad_sch (KiCad schematic)
At the start: 8 parts, among them J1 Conn_02x10_Odd_Even, U1 DRV8837C, U2 TPL7407LA, U3 74AHCT1G04, U4 TPL7407LA

Commit message: Start IO schematic
Parts:
- removed C1, C2, C3: 0u1, symbol Device:C
- removed U1: DRV8837C, Package_SON:WSON-8-1EP_2x2mm_P0.5mm_EP0.9x1.6mm, symbol Driver_Motor:DRV8837C
- removed U3: 74AHCT1G04, symbol 74xGxx:74AHCT1G04
- added C4, C5: 0u1, Capacitor_SMD:C_0603_1608Metric_Pad1.08x0.95mm_HandSolder, symbol Device:C
- added J2: Conn_01x02_Socket, symbol Connector:Conn_01x02_Socket
- added R10, R11, R12, R13, R2, R3, R4, R5, R6, R7, R8, R9: 100k, Resistor_SMD:R_0603_1608Metric_Pad0.98x0.95mm_HandSolder, symbol Device:R
- added U5: TCA9535PWR, Package_SO:TSSOP-24_4.4x7.8mm_P0.65mm, symbol Interface_Expansion:TCA9535PWR
- added U6: OPT4048, symbol Global:OPT4048
- J1: footprint (none) -> Connector_IDC:IDC-Header_2x10_P2.54mm_Vertical
Connections:
- net LATCH is gone; now on net GND: J1.2 (Pin_2)
- net SW0 is gone; now on net GND: J1.10 (Pin_10)
- net SW6 is gone; now on net AIN1: J1.16 (Pin_16)
- net nEN is gone; now on net GND: J1.5 (Pin_5)
- net +3V3: now also C4.1, C5.1, U5.24 (VCC), U6.1 (Vdd), U6.2 (ADDR)
- net +5V: now also J1.6 (Pin_6)
- net +VSW: now also U2.9 (COM), U4.9 (COM), R10.2, R11.2, R12.2, R13.2, R2.2, R3.2, R4.2, R5.2, R6.2, R7.2, R8.2, R9.2
- net AIN1: no longer J1.20 (Pin_20)
- net GND: now also U2.8 (GND), U4.6 (I6), U4.7 (I7), U4.8 (GND), C4.2, C5.2, U5.12 (GND), U5.2 (A1), U5.21 (A0), U5.3 (A2), U6.4 (GND); no longer J1.17 (Pin_17), J1.19 (Pin_19), J1.6 (Pin_6)
- net 1: now reaches U4.1 (I1)
- net 1: now also U5.11 (P07)
- net at U4.12 (O5): now also R13.1
- net at U4.13 (O4): now also R12.1
- net at U4.14 (O3): now also R11.1
- net at U4.15 (O2): now also R10.1
- net at U4.16 (O1): now also R9.1
- net 2: now reaches U4.2 (I2)
- net 2: now also U5.13 (P10)
- net 3: now reaches U4.3 (I3)
- net 3: now also U5.14 (P11)
- net 4: now reaches U4.4 (I4)
- net 4: now also U5.15 (P12)
- net sep: now reaches U4.5 (I5)
- net sep: now also U5.16 (P13)
- net a: now reaches U2.1 (I1)
- net a: now also U5.4 (P00)
- net at U2.10 (O7): now also R8.1
- net at U2.11 (O6): now also R7.1
- net at U2.12 (O5): now also R6.1
- net at U2.13 (O4): now also R5.1
- net at U2.14 (O3): now also R4.1
- net at U2.15 (O2): now also R3.1
- net at U2.16 (O1): now also R2.1
- net b: now reaches U2.2 (I2)
- net b: now also U5.5 (P01)
- net c: now reaches U2.3 (I3)
- net c: now also U5.6 (P02)
- net d: now reaches U2.4 (I4)
- net d: now also U5.7 (P03)
- net e: now reaches U2.5 (I5)
- net e: now also U5.8 (P04)
- net f: now reaches U2.6 (I6)
- net f: now also U5.9 (P05)
- net g: now reaches U2.7 (I7)
- net g: now also U5.10 (P06)
- net AIN0 renamed AIN2
- net CLK renamed I2C_SDA
- net I2C_SDA: now also U5.23 (SDA), U6.8 (SDA)
- net DAT renamed I2C_SCL
- net I2C_SCL: now also U5.22 (SCL), U6.5 (SCL)
- net PWM: no longer names the net of J1.4 (Pin_4)
- net SW1 renamed SWI1
- net SW2 renamed SWI2
- net SW3 renamed SWI3
- net SW4 renamed SWI4
- net SW5 renamed Vref
- new net AIN3: J1.17 (Pin_17)
- new net Audio+: J1.19 (Pin_19), J2.1 (Pin_1)
- new net Audio-: J1.20 (Pin_20), J2.2 (Pin_2)
- new net disp_En: U5.17 (P14)
- no-connect marks 0 -> 4
Other:
- added sheet Buttons (buttons.kicad_sch)
- added sheet Filament Drive (filament.kicad_sch)
- sheet VFD Power ports: added 5Vin, EN, SCL, SDA; removed Vin
- moved on the sheet: U2, U4

Commit message: Update IO Board
Parts:
- J2: footprint (none) -> Connector_PinHeader_2.54mm:PinHeader_1x02_P2.54mm_Vertical
- U6: footprint (none) -> kicad global library:SOT-583_DTS
Connections:
- net a: now also U2.7 (I7); no longer U2.1 (I1)
- net b: now also U2.6 (I6); no longer U2.2 (I2)
- net c: now also U2.5 (I5); no longer U2.3 (I3)
- net e: now also U2.3 (I3); no longer U2.5 (I5)
- net f: now also U2.2 (I2); no longer U2.6 (I6)
- net g: now also U2.1 (I1); no longer U2.7 (I7)
- net c_HV: now reaches R6.1, U2.12 (O5)
- net sep_HV: now reaches R13.1, U4.12 (O5)
- net 3_HV: now reaches R11.1, U4.14 (O3)
- net 1_HV: now reaches R9.1, U4.16 (O1)
- net 4_HV: now reaches R12.1, U4.13 (O4)
- net 2_HV: now reaches R10.1, U4.15 (O2)
- net a_HV: now reaches R8.1, U2.10 (O7)
- net b_HV: now reaches R7.1, U2.11 (O6)
- net d_HV: now reaches R5.1, U2.13 (O4)
- net e_HV: now reaches R4.1, U2.14 (O3)
- net f_HV: now reaches R3.1, U2.15 (O2)
- net g_HV: now reaches R2.1, U2.16 (O1)
Changed lines of the file:
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@@
 	)
 	(label "g"
-		(at 261.62 92.71 180)
+		(at 261.62 77.47 180)
 		(fields_autoplaced yes)
 		(effects
@@
 		)
 	)
+	(label "4_HV"
+		(at 317.5 128.27 0)
+		(fields_autoplaced yes)
+		(effects
+			(font
+				(size 1.27 1.27)
+			)
+			(justify left bottom)
+		)
+	)
+	(label "sep_HV"
+		(at 327.66 130.81 0)
+		(fields_autoplaced yes)
+		(effects
+			(font
+				(size 1.27 1.27)
+			)
+			(justify left bottom)
+		)
+	)
 	(label "f"
-		(at 261.62 90.17 180)
+		(at 261.62 80.01 180)
 		(fields_autoplaced yes)
 		(effects
@@
 	)
 	(label "a"
-		(at 261.62 77.47 180)
+		(at 261.62 92.71 180)
 		(fields_autoplaced yes)
 		(effects
@@
 	)
 	(label "b"
-		(at 261.62 80.01 180)
+		(at 261.62 90.17 180)
 		(fields_autoplaced yes)
 		(effects
@@
 		)
 	)
+	(label "3_HV"
+		(at 307.34 125.73 0)
+		(fields_autoplaced yes)
+		(effects
+			(font
+				(size 1.27 1.27)
+			)
+			(justify left bottom)
+		)
+	)
 	(label "SWI2"
 		(at 54.61 135.89 180)
@@
 		)
 	)
+	(label "b_HV"
+		(at 337.82 90.17 0)
+		(fields_autoplaced yes)
+		(effects
+			(font
+				(size 1.27 1.27)
+			)
+			(justify left bottom)
+		)
+	)
 	(label "Audio-"
 		(at 53.34 49.53 0)
@@
 		)
 	)
+	(label "c_HV"
+		(at 327.66 87.63 0)
+		(fields_autoplaced yes)
+		(effects
+			(font
+				(size 1.27 1.27)
+			)
+			(justify left bottom)
+		)
+	)
 	(label "AIN2"
 		(at 53.34 46.99 0)
@@
 		)
 	)
+	(label "g_HV"
+		(at 287.02 77.47 0)
+		(fields_autoplaced yes)
+		(effects
+			(font
+				(size 1.27 1.27)
+			)
+			(justify left bottom)
+		)
+	)
+	(label "f_HV"
+		(at 297.18 80.01 0)
+		(fields_autoplaced yes)
+		(effects
+			(font
+				(size 1.27 1.27)
+			)
+			(justify left bottom)
+		)
+	)
 	(label "AIN1"
 		(at 54.61 143.51 180)
@@
 		)
 	)
+	(label "e_HV"
+		(at 307.34 82.55 0)
+		(fields_autoplaced yes)
+		(effects
+			(font
+				(size 1.27 1.27)
+			)
+			(justify left bottom)
+		)
+	)
 	(label "VFa"
 		(at 140.97 229.87 0)
@@
 		)
 	)
+	(label "a_HV"
+		(at 347.98 92.71 0)
+		(fields_autoplaced yes)
+		(effects
+			(font
+				(size 1.27 1.27)
+			)
+			(justify left bottom)
+		)
+	)
 	(label "2"
 		(at 144.78 66.04 0)
@@
 		)
 	)
+	(label "d_HV"
+		(at 317.5 85.09 0)
+		(fields_autoplaced yes)
+		(effects
+			(font
+				(size 1.27 1.27)
+			)
+			(justify left bottom)
+		)
+	)
 	(label "sep"
 		(at 261.62 130.81 180)
@@
 		)
 	)
+	(label "1_HV"
+		(at 287.02 120.65 0)
+		(fields_autoplaced yes)
+		(effects
+			(font
+				(size 1.27 1.27)
+			)
+			(justify left bottom)
+		)
+	)
 	(label "g"
 		(at 144.78 58.42 0)
@@
 		)
 	)
+	(label "2_HV"
+		(at 297.18 123.19 0)
+		(fields_autoplaced yes)
+		(effects
+			(font
+				(size 1.27 1.27)
+			)
+			(justify left bottom)
+		)
+	)
 	(label "I2C_SDA"
 		(at 109.22 43.18 180)
@@
 	)
 	(label "e"
+		(at 261.62 82.55 180)
+		(fields_autoplaced yes)
+		(effects
+			(font
+				(size 1.27 1.27)
+			)
+			(justify right bottom)
+		)
+	)
+	(label "c"
 		(at 261.62 87.63 180)
-		(fields_autoplaced yes)
-		(effects
-			(font
-				(size 1.27 1.27)
-			)
-			(justify right bottom)
-		)
-	)
-	(label "c"
-		(at 261.62 82.55 180)
 		(fields_autoplaced yes)
 		(effects
@@
 			)
 		)
-		(property "Footprint" ""
+		(property "Footprint" "Connector_PinHeader_2.54mm:PinHeader_1x02_P2.54mm_Vertical"
 			(at 50.8 62.23 0)
 			(effects
@@
 			)
 		)
-		(property "Footprint" ""
+		(property "Footprint" "kicad global library:SOT-583_DTS"
 			(at 137.16 133.35 0)
 			(effects

Commit message: Update IO board
Parts:
- removed R10, R11, R12, R13, R2, R3, R4, R5, R6, R7, R8, R9: 100k, Resistor_SMD:R_0603_1608Metric_Pad0.98x0.95mm_HandSolder, symbol Device:R
- removed U2, U4: TPL7407LA, Package_SO:TSSOP-16_4.4x5mm_P0.65mm, symbol Global:TPL7407LA
- removed U5: TCA9535PWR, Package_SO:TSSOP-24_4.4x7.8mm_P0.65mm, symbol Interface_Expansion:TCA9535PWR
- added C14: 0u1, Capacitor_SMD:C_0603_1608Metric_Pad1.08x0.95mm_HandSolder, symbol Device:C
- added C15, C16, C17, C18: 0u1, 50V, Capacitor_SMD:C_0603_1608Metric_Pad1.08x0.95mm_HandSolder, symbol Device:C
- added H1, H2, H3, H4: MountingHole_Pad, MountingHole:MountingHole_3.2mm_M3_Pad, symbol Mechanical:MountingHole_Pad
- added R1: 10k, Resistor_SMD:R_0603_1608Metric_Pad0.98x0.95mm_HandSolder, symbol Device:R
- added R17: 470R, Resistor_SMD:R_0603_1608Metric_Pad0.98x0.95mm_HandSolder, symbol Device:R
- added U11, U12, U2, U4: TLV1824, kicad global library:SOT-23-THIN-14_2x4.2mm_P0.5_TI-DYY_HandSoldering, symbol Global:TLV1824
- added U13: TCA9555PWR, Package_SO:TSSOP-24_4.4x7.8mm_P0.65mm, symbol Interface_Expansion:TCA9555PWR
- added VFD1: IVL2-7/5, kicad global library:IVL2-75, symbol Global:IVL2-7/5
Connections:
- net +3V3: now also U13.24 (VCC)
- net +VSW: now also C15.1, C16.1, C17.1, C18.1, U11.3 (V+), U12.3 (V+), U2.3 (V+), U4.3 (V+)
- net 1: now also U11.7 (+), U13.14 (P11)
- net 1_HV: now also U11.1, VFD1.2 (K1), VFD1.22 (K1)
- net 2: now also U11.9 (+), U13.15 (P12)
- net 2_HV: now also U11.14, VFD1.21 (K2), VFD1.6 (K2)
- net 3: now also U11.11 (+), U13.16 (P13)
- net 3_HV: now also U11.13, VFD1.11 (K4), VFD1.19 (K4)
- net 4: now also U12.5 (+), U13.17 (P14)
- net 4_HV: now also U12.2, VFD1.15 (K5), VFD1.18 (K5)
- net GND: now also J1.4 (Pin_4), C14.2, C15.2, C16.2, C17.2, C18.2, H1.1, H2.1, H3.1, H4.1, R1.2, U11.12 (V-), U12.11 (+), U12.12 (V-), U12.9 (+), U13.12 (GND), U13.2 (A1), U13.21 (A0), U13.3 (A2), U2.12 (V-), U4.12 (V-)
- net I2C_SCL: now also U13.22 (SCL)
- net I2C_SDA: now also U13.23 (SDA)
- net VFa: now also VFD1.1 (F1), VFD1.23 (F1)
- net VFb: now also VFD1.16 (F2), VFD1.17 (F2)
- net Vref: now also R17.2
- net a: now also U13.4 (P00), U2.5 (+)
- net a_HV: now also U2.2, VFD1.14 (a)
- net b: now also U13.5 (P01), U2.7 (+)
- net b_HV: now also U2.1, VFD1.12 (b)
- net c: now also U13.6 (P02), U2.9 (+)
- net c_HV: now also U2.14, VFD1.7 (c)
- net d: now also U13.7 (P03), U2.11 (+)
- net d_HV: now also U2.13, VFD1.10 (d)
- net disp_En: now also R1.1, U13.19 (P16)
- net e: now also U13.8 (P04), U4.5 (+)
- net e_HV: now also U4.2, VFD1.5 (e)
- net f: now also U13.9 (P05), U4.7 (+)
- net f_HV: now also U4.1, VFD1.13 (f)
- net g: now also U13.10 (P06), U4.9 (+)
- net g_HV: now also U4.14, VFD1.4 (g)
- net sep: now also U12.7 (+), U13.18 (P15)
- net sep_HV: now also U12.1, VFD1.20 (K3), VFD1.8 (K3)
- new net COMP_REF: C14.1, R17.1, U11.10 (-), U11.4 (-), U11.6 (-), U11.8 (-), U12.10 (-), U12.4 (-), U12.6 (-), U12.8 (-), U2.10 (-), U2.4 (-), U2.6 (-), U2.8 (-), U4.10 (-), U4.4 (-), U4.6 (-), U4.8 (-)
- new net sep_bottom: U11.5 (+), U13.13 (P10)
- new net sep_bottom_HV: U11.2, VFD1.9 (s_b)
- new net sep_top: U13.11 (P07), U4.11 (+)
- new net sep_top_HV: U4.13, VFD1.3 (s_t)
- no-connect marks 4 -> 5
