File: Alarm IO Board/filament.kicad_sch (KiCad schematic)
At the start: 9 parts, among them U1 74AHCT1G04, U3 DRV8837C, U8 TPS7A0525PDBV

Commit message: Update IO Board
Parts:
- removed C2: 0u1, symbol Device:C
- removed U1: 74AHCT1G04, symbol 74xGxx:74AHCT1G04
- added C10: 18p, Capacitor_SMD:C_0603_1608Metric_Pad1.08x0.95mm_HandSolder, symbol Device:C
- added C11, C12: 0u1, Capacitor_SMD:C_0603_1608Metric_Pad1.08x0.95mm_HandSolder, symbol Device:C
- added R14: 330k, Resistor_SMD:R_0603_1608Metric_Pad0.98x0.95mm_HandSolder, symbol Device:R
- added U1, U9: SN74LVC1G132, Package_TO_SOT_SMD:SOT-23-5, symbol Global:SN74LVC1G132
- C1, C3: footprint (none) -> Capacitor_SMD:C_0603_1608Metric_Pad1.08x0.95mm_HandSolder
- U3: footprint Package_SON:WSON-8-1EP_2x2mm_P0.5mm_EP0.9x1.6mm -> kicad global library:WSON-8-1EP_2x2mm_P0.5mm_EP0.9x1.6mm_HandSoldering
Connections:
- net 3Vin: now also C11.1, C12.1, U1.5 (VCC), U9.5 (VCC)
- net EN: now also U1.2 (B), U9.1 (A)
- net GND: now also C10.2, C11.2, C12.2, U1.3 (GND), U9.3 (GND)
- net VFD_Fil_SWA: now also R14.1, U1.4 (Y), U9.2 (B)
- net VFD_Fil_SWB: now also U9.4 (Y)
- new net: C10.1, R14.2, U1.1 (A)
Other:
- note added: "Rough RC Oscillator (~100kHz)"

Commit message: Update IO board
Parts:
- removed R1: 10k, Resistor_SMD:R_0603_1608Metric_Pad0.98x0.95mm_HandSolder, symbol Device:R
Changed lines of the file:
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@@
-	)
-	(junction
-		(at 111.76 81.28)
-		(diameter 0)
-		(color 0 0 0 0)
 	)
 	(junction
@@
 	(wire
 		(pts
-			(xy 111.76 81.28) (xy 133.35 81.28)
-		)
-		(stroke
-			(width 0)
-			(type default)
-		)
-	)
-	(wire
-		(pts
 			(xy 43.18 106.68) (xy 78.74 106.68)
 		)
@@
 	(wire
 		(pts
-			(xy 106.68 81.28) (xy 111.76 81.28)
+			(xy 106.68 81.28) (xy 133.35 81.28)
 		)
 		(stroke
@@
 		)
 	)
-	(symbol
-		(lib_id "Device:R")
-		(at 111.76 85.09 0)
-		(unit 1)
-		(exclude_from_sim no)
-		(in_bom yes)
-		(on_board yes)
-		(dnp no)
-		(fields_autoplaced yes)
-		(property "Reference" "R1"
-			(at 114.3 83.8199 0)
-			(effects
-				(font
-					(size 1.27 1.27)
-				)
-				(justify left)
-			)
-		)
-		(property "Value" "10k"
-			(at 114.3 86.3599 0)
-			(effects
-				(font
-					(size 1.27 1.27)
-				)
-				(justify left)
-			)
-		)
-		(property "Footprint" "Resistor_SMD:R_0603_1608Metric_Pad0.98x0.95mm_HandSolder"
-			(at 109.982 85.09 90)
-			(effects
-				(font
-					(size 1.27 1.27)
-				)
-				(hide yes)
-			)
-		)
-		(property "Datasheet" "~"
-			(at 111.76 85.09 0)
-			(effects
-				(font
-					(size 1.27 1.27)
-				)
-				(hide yes)
-			)
-		)
-		(property "Description" "Resistor"
-			(at 111.76 85.09 0)
-			(effects
-				(font
-					(size 1.27 1.27)
-				)
-				(hide yes)
-			)
-		)
-		(pin "2"
-		)
-		(pin "1"
-		)
-		(instances
-			(project "Alarm IO Board"
-				(path "/1724f6e0-4b54-44f9-83c3-b4b5d1121f36/4343f827-c32e-4b41-8108-6356139d2572"
-					(reference "R1")
-					(unit 1)
-				)
-			)
-		)
-	)
-	(symbol
-		(lib_id "power:GND")
-		(at 111.76 88.9 0)
-		(unit 1)
-		(exclude_from_sim no)
-		(in_bom yes)
-		(on_board yes)
-		(dnp no)
-		(fields_autoplaced yes)
-		(property "Reference" "#PWR027"
-			(at 111.76 95.25 0)
-			(effects
-				(font
-					(size 1.27 1.27)
-				)
-				(hide yes)
-			)
-		)
-		(property "Value" "GND"
-			(at 111.76 93.98 0)
-			(effects
-				(font
-					(size 1.27 1.27)
-				)
-			)
-		)
-		(property "Footprint" ""
-			(at 111.76 88.9 0)
-			(effects
-				(font
-					(size 1.27 1.27)
-				)
-				(hide yes)
-			)
-		)
-		(property "Datasheet" ""
-			(at 111.76 88.9 0)
-			(effects
-				(font
-					(size 1.27 1.27)
-				)
-				(hide yes)
-			)
-		)
-		(property "Description" "Power symbol creates a global label with name \"GND\" , ground"
-			(at 111.76 88.9 0)
-			(effects
-				(font
-					(size 1.27 1.27)
-				)
-				(hide yes)
-			)
-		)
-		(pin "1"
-		)
-		(instances
-			(project "Alarm IO Board"
-				(path "/1724f6e0-4b54-44f9-83c3-b4b5d1121f36/4343f827-c32e-4b41-8108-6356139d2572"
-					(reference "#PWR027")
-					(unit 1)
-				)
-			)
-		)
-	)
